File: v2/pcb/business_card_v1.brd (EAGLE design)
At the start: 89 x 51 mm, 75 parts, among them SW1 SPST_TACT-KMR2

Commit message: get the businss card completed
Parts:
- C1: device adafruit:C0603K -> rcl:C0805
- R1, R2, R3, R4, R5, R6, R7, R8, R9: device resistor:R0603 -> rcl:R0805
- moved SW1 0.63 mm to (33.0, 6.99)
Routing:
- net GND: track 11.6 -> 14.1 mm, vias 4 -> 3
- net RESET: track 13.2 -> 13.7 mm
