File: v2/business_card_pcb/business_card_v1.brd (EAGLE design)
At the start: 89 x 51 mm, 75 parts, among them SW1 SPST_TACT-KMR2

Commit message: get the published version completed
Parts:
- moved U$1 0.63 mm to (5.08, 45.7)
Routing:
- net GND: track 13.2 -> 14.0 mm, vias 3 -> 2
Other:
- board text added: "Plug the USB connector into any USB port, and watch the LED display. Project details can be found at github.com/kevinlutzer/business-card"
- board text added: "Website: kevin.lutzer.ca Email: kevin@lutzer.ca Github: github.com/kevinlutzer LinkedIn: linkedin.com/in/kevin-lutzer"
- board text removed: "Plug the usb connector into any usb port, and watch the LED display. Project details can be found at https://bit.ly/38gpalY"
- board text removed: "Website: kevin.lutzer.ca Email: kevin@lutzer.ca Github: github.com/kevinlutzer Linkedin: linkedin.com/in/kevin-lutzer"
Changed lines of the file:
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@@
 <drawing>
 <settings>
-<setting alwaysvectorfont="yes"/>
+<setting alwaysvectorfont="no"/>
 <setting verticaltext="up"/>
 </settings>
@@
 <layer number="30" name="bStop" color="7" fill="6" visible="no" active="yes"/>
 <layer number="31" name="tCream" color="7" fill="4" visible="no" active="yes"/>
-<layer number="32" name="bCream" color="7" fill="5" visible="no" active="yes"/>
+<layer number="32" name="bCream" color="7" fill="5" visible="yes" active="yes"/>
 <layer number="33" name="tFinish" color="6" fill="3" visible="no" active="yes"/>
 <layer number="34" name="bFinish" color="6" fill="6" visible="no" active="yes"/>
@@
 <wire x1="89" y1="0" x2="89" y2="51" width="0" layer="20"/>
 <wire x1="89" y1="51" x2="0" y2="51" width="0" layer="20"/>
-<text x="8.89" y="47.625" size="1.27" layer="25">v2</text>
-<text x="8.89" y="44.45" size="2.54" layer="25">Kevin Lutzer</text>
-<text x="2.54" y="39.37" size="1.778" layer="25">B.E. Electrical Engineering &amp;
+<text x="8.255" y="46.99" size="1.27" layer="25">v2</text>
+<text x="8.255" y="43.815" size="2.54" layer="25">Kevin Lutzer</text>
+<text x="2.54" y="38.1" size="1.778" layer="25">B.E. Electrical Engineering &amp;
 B.Sc. Computer Science</text>
-<text x="2.54" y="28.575" size="1.778" layer="25">Website: kevin.lutzer.ca
+<text x="2.54" y="27.305" size="1.778" layer="25">Website: kevin.lutzer.ca
 Email: kevin@lutzer.ca
 Github: github.com/kevinlutzer
-Linkedin: linkedin.com/in/kevin-lutzer</text>
-<text x="45.72" y="38.735" size="1.778" layer="26" rot="MR0">Plug the usb connector into any usb
+LinkedIn: linkedin.com/in/kevin-lutzer</text>
+<text x="45.72" y="38.735" size="1.778" layer="26" rot="MR0">Plug the USB connector into any USB
 port, and watch the LED display.
 Project details can be found at
-https://bit.ly/38gpalY</text>
+github.com/kevinlutzer/business-card</text>
 <wire x1="0.01081875" y1="0.00856875" x2="0.01073125" y2="0.008740625" width="0.025" layer="121"/>
 <wire x1="0.01073125" y1="0.008740625" x2="0.0104" y2="0.009209375" width="0.025" layer="121"/>
@@
 <attribute name="VALUE" x="38.6715" y="12.3825" size="1.27" layer="27" ratio="10" rot="R270"/>
 </element>
-<element name="U$1" library="adafruit" library_urn="urn:adsk.eagle:library:420" package="OSHWLOGO_TOP_0.2" package3d_urn="urn:adsk.eagle:package:6240813/1" override_package3d_urn="urn:adsk.eagle:package:17231582/2" override_package_urn="urn:adsk.eagle:footprint:6240168/1" value="" x="5.08" y="46.355" smashed="yes"/>
+<element name="U$1" library="adafruit" library_urn="urn:adsk.eagle:library:420" package="OSHWLOGO_TOP_0.2" package3d_urn="urn:adsk.eagle:package:6240813/1" override_package3d_urn="urn:adsk.eagle:package:17231582/2" override_package_urn="urn:adsk.eagle:footprint:6240168/1" value="" x="5.08" y="45.72" smashed="yes"/>
 <element name="TP1" library="SparkFun-Connectors" package="1X01_NO_SILK" value="TEST-POINTPOGO_PTH" x="29.21" y="8.255" smashed="yes"/>
-<element name="TP2" library="SparkFun-Connectors" package="1X01_NO_SILK" value="TEST-POINTPOGO_PTH" x="29.21" y="3.175" smashed="yes">
-<attribute name="VALUE" x="27.94" y="1.397" size="0.6096" layer="27" font="vector" ratio="20"/>
-</element>
+<element name="TP2" library="SparkFun-Connectors" package="1X01_NO_SILK" value="TEST-POINTPOGO_PTH" x="29.21" y="3.175" smashed="yes"/>
 <element name="TP3" library="SparkFun-Connectors" package="1X01_NO_SILK" value="TEST-POINTPOGO_PTH" x="29.21" y="13.335" smashed="yes"/>
 <element name="TP4" library="SparkFun-Connectors" package="1X01_NO_SILK" value="TEST-POINTPOGO_PTH" x="29.21" y="5.715" smashed="yes"/>
@@
 <wire x1="40.955" y1="15.24" x2="42.545" y2="15.24" width="0.3048" layer="1"/>
 <via x="42.545" y="15.24" extent="1-16" drill="0.35"/>
-<wire x1="42.6085" y1="12.7" x2="44.45" y2="12.7" width="0.3048" layer="1"/>
-<via x="44.45" y="12.7" extent="1-16" drill="0.35"/>
 <contactref element="TP5" pad="1"/>
 <contactref element="SW1" pad="4"/>
@@
 <wire x1="9.525" y1="14.474746875" x2="9.525" y2="14.605" width="0.6096" layer="1"/>
 <via x="9.525" y="14.605" extent="1-16" drill="0.35"/>
+<wire x1="42.545" y1="12.7" x2="42.545" y2="15.24" width="0.3048" layer="1"/>
+<wire x1="42.6085" y1="12.7" x2="42.545" y2="12.7" width="0.3048" layer="1"/>
 </signal>
 <signal name="UCC">
@@
 <wire x1="10.28345" y1="5.333703125" x2="15.744746875" y2="10.795" width="0.6096" layer="1"/>
 <wire x1="15.744746875" y1="10.795" x2="15.875" y2="10.795" width="0.6096" layer="1"/>
-<wire x1="15.875" y1="10.795" x2="15.875" y2="10.16" width="0.6096" layer="1"/>
+<wire x1="15.875" y1="10.16" x2="15.875" y2="10.795" width="0.6096" layer="1"/>
 </signal>
 <signal name="RESET">
