File: v3/_autosave-business_card_v1.kicad_pcb (KiCad board)
At the start: 16 copper layers, 89 x 51 mm, 67 parts, among them J1 Conn_01x05_Male, SW1 SPST_TACT-KMR2, U1 MIC5504-3.3YM5, U2 STM32G030F6P6

Commit message: finish pcb prototype for the card
Routing:
- net SWDCLK-BOOT0: track 11.4 -> 17.2 mm
Changed lines of the file:
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@@
     (thickness 1.6)
     (drawings 236)
-    (tracks 415)
+    (tracks 416)
     (zones 0)
     (modules 67)
@@
   (segment (start 141.0225 126.5665) (end 141.0225 127.513) (width 0.25) (layer Top) (net 22))
   (segment (start 141.351 126.238) (end 141.0225 126.5665) (width 0.25) (layer Top) (net 22))
-  (segment (start 136.289999 122.243053) (end 136.289999 119.652999) (width 0.25) (layer Bottom) (net 22))
-  (segment (start 136.289999 119.652999) (end 135.89 119.253) (width 0.25) (layer Bottom) (net 22))
-  (segment (start 140.673599 125.560599) (end 139.607545 125.560599) (width 0.25) (layer Bottom) (net 22))
-  (segment (start 141.351 126.238) (end 140.673599 125.560599) (width 0.25) (layer Bottom) (net 22))
   (segment (start 132.207 119.253) (end 132.08 119.126) (width 0.25) (layer Top) (net 22))
   (segment (start 135.89 119.253) (end 132.207 119.253) (width 0.25) (layer Top) (net 22))
+  (segment (start 137.752599 125.560599) (end 140.673599 125.560599) (width 0.25) (layer Bottom) (net 22))
+  (segment (start 136.289999 124.097999) (end 137.752599 125.560599) (width 0.25) (layer Bottom) (net 22))
+  (segment (start 140.673599 125.560599) (end 141.351 126.238) (width 0.25) (layer Bottom) (net 22))
+  (segment (start 136.289999 119.652999) (end 136.289999 124.097999) (width 0.25) (layer Bottom) (net 22))
+  (segment (start 135.89 119.253) (end 136.289999 119.652999) (width 0.25) (layer Bottom) (net 22))
   (zone (net 11) (net_name +3V3) (layer Top) (hatch edge 0.508)
     (connect_pads (clearance 0.508))
