File: v3/business-card-v3-pcb/business-card-v3-programmer-board-pcb/business-card-v3-programmer-board-pcb.kicad_pcb (KiCad board)
At the start: 2 copper layers, 100 x 100 mm, 17 parts, among them J1 Pogo_Pin_Conn, J2 Power_TP, J3 Programmer_Conn, J4 Jack-DC, SW1 RST, U1 LM2904, U2 L7805CV

Commit message: finish the pcb design
Parts:
- moved J1 23.5 mm to (130.6, 122.2)
- moved J2 16.2 mm to (121.0, 122.2)
- turned H1 to 180 degrees
- turned H3 to 180 degrees
Routing:
- net RST: track 0.00 -> 107.9 mm
- net +3V3: track 0.00 -> 102.1 mm
- net SWDIO: track 0.00 -> 68.9 mm
- net SWCLK: track 0.00 -> 63.3 mm
- net GND: track 16.9 -> 18.1 mm
Other:
- board text added: "Business_Card_V1"
