File: v3/business-card-v3-pcb/business-card-v3-programmer-board-pcb/business-card-v3-programmer-board-pcb.sch (KiCad schematic (older format))
At the start: 17 parts, among them J1 Pogo_Pin_Conn, J2 Power_TP, J3 Programmer_Conn, J4 Jack-DC, SW1 RST, U1 LM2904, U2 L7805CV

Commit message: finish the pcb design
Other:
- note added: "3.3V VREF Tester"
- note added: "Mounting Holes"
- note added: "Power Supply"
- note added: "Test Points and Programmer\nHeaders"
- moved on the sheet: C1, C2, D1, D2, H1, H2, H3, H4, J1, J2, J3, J4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
