File: v3/business-card-v3-pcb/business_card_v1.sch (KiCad schematic (older format))
At the start: 68 parts, among them J1 Conn_01x05_Male, J2 Conn_01x01_Male, SW1 SW_SPST, U1 MIC5504-3.3YM5, U2 STM32G030F6P6

Commit message: update to use a smaller resistor array
Parts:
- RN1, RN2: footprint Resistor_SMD:R_Array_Convex_4x1206 -> Resistor_SMD:R_Array_Convex_4x0603
Changed lines of the file:
@@
 F 0 "RN1" V 5283 5500 50  0000 C CNN
 F 1 "R_Pack04" V 5374 5500 50  0000 C CNN
-F 2 "Resistor_SMD:R_Array_Convex_4x1206" V 5975 5500 50  0001 C CNN
+F 2 "Resistor_SMD:R_Array_Convex_4x0603" V 5975 5500 50  0001 C CNN
 F 3 "~" H 5700 5500 50  0001 C CNN
 	1    5700 5500
@@
 F 0 "RN2" V 9200 5500 50  0000 C CNN
 F 1 "R_Pack04" V 9100 5500 50  0000 C CNN
-F 2 "Resistor_SMD:R_Array_Convex_4x1206" V 9175 5500 50  0001 C CNN
+F 2 "Resistor_SMD:R_Array_Convex_4x0603" V 9175 5500 50  0001 C CNN
 F 3 "~" H 8900 5500 50  0001 C CNN
 	1    8900 5500
