File: pcb/business_card.kicad_sch (KiCad schematic)
At the start: 68 parts, among them J3 USB_A, J4 Conn_ARM_SWD_TagConnect_TC2030, SW1 SW_SPST, U1 MIC5504-3.3YM5, U2 STM32G030F6P6

Commit message: remove the progremmwer and the eagle files, rename everything to just business card
Parts:
- LED1, LED2: value LEDCHIPLED_0805 -> LED
Changed lines of the file:
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@@
       (effects (font (size 1.4986 1.4986)) (justify left bottom))
     )
-    (property "Value" "LEDCHIPLED_0805" (at 146.685 25.908 90)
+    (property "Value" "LED" (at 146.685 25.908 90)
       (effects (font (size 1.4986 1.4986)) (justify left bottom) hide)
     )
@@
       (effects (font (size 1.4986 1.4986)) (justify left bottom))
     )
-    (property "Value" "LEDCHIPLED_0805" (at 126.365 25.908 90)
+    (property "Value" "LED" (at 126.365 25.908 90)
       (effects (font (size 1.4986 1.4986)) (justify left bottom) hide)
     )

Commit message: use leds instead, add bom, update code
Parts:
- D1, D10, D11, D12, D13, D14, D15, D16, D17, D18, D19, D2, D20, D21, D22, D23, D24, D25, D26, D27, D28, D29, D3, D30, D31, D32, D33, D34, D35, D36, D37, D38, D39, D4, D40, D41, D42, D43, D44, D45, D46, D47, D48, D49, D5, D50, D51, D52, D53, D54, D6, D7, D8, D9, LED1: footprint Diode_SMD:D_0805_2012Metric -> LED_SMD:LED_0805_2012Metric

Commit message: use the LED footprint instead of diode footprint for LED2
Parts:
- LED2: footprint Diode_SMD:D_0805_2012Metric -> LED_SMD:LED_0805_2012Metric
Changed lines of the file:
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@@
       (effects (font (size 1.4986 1.4986)) (justify left bottom) hide)
     )
-    (property "Footprint" "Diode_SMD:D_0805_2012Metric" (at 152.4 30.48 0)
+    (property "Footprint" "LED_SMD:LED_0805_2012Metric" (at 152.4 30.48 0)
       (effects (font (size 1.27 1.27)) hide)
     )
